Commit message: Using macros for new_leg.xacro

File: qronk_description/urdf/new_leg.xacro (robot description, xacro)
@@ -3,24 +3,5 @@
 <xacro:include filename="$(find qronk_description)/urdf/materials.xacro" />
 <xacro:include filename="$(find qronk_description)/urdf/new_leg.trans" />
-<link name="base_link">
-  <inertial>
-    <origin xyz="2.8303654344169608e-18 -3.5112443987378646e-18 0.0009999999999999994" rpy="0 0 0"/>
-    <mass value="0.030826877913349836"/>
-    <inertia ixx="5e-06" iyy="5e-06" izz="1e-05" ixy="-0.0" iyz="-0.0" ixz="0.0"/>
-  </inertial>
-  <visual>
-    <origin xyz="0 0 0" rpy="0 0 0"/>
-    <geometry>
-      <mesh filename="package://qronk_description/meshes/base_link.stl" scale="0.001 0.001 0.001"/>
-    </geometry>
-    <material name="steel_satin"/>
-  </visual>
-  <collision>
-    <origin xyz="0 0 0" rpy="0 0 0"/>
-    <geometry>
-      <mesh filename="package://qronk_description/meshes/base_link.stl" scale="0.001 0.001 0.001"/>
-    </geometry>
-  </collision>
-</link>
+<xacro:macro name="leg" params="side">
 <link name="SHORT_DRIVER_v3_1">
   <inertial>
@@ -103,29 +84,32 @@
   </collision>
 </link>
-<joint name="A" type="continuous">
+<joint name="${side}_upper_leg" type="revolute">
   <origin xyz="0.0 0.0 0.002" rpy="0 0 0"/>
-  <parent link="base_link"/>
+  <parent link="chassis"/>
   <child link="SHORT_DRIVER_v3_1"/>
   <axis xyz="0.0 -0.0 1.0"/>
+  <limit effort="1000.0" lower="${pi}" upper="${-pi}" velocity="100"/>
 </joint>
-<joint name="B" type="continuous">
+<joint name="${side}_lower_leg" type="revolute">
   <origin xyz="-0.031 0.0 0.005" rpy="0 0 0"/>
   <parent link="SHORT_DRIVER_v3_1"/>
   <child link="INNER_BAR_v4_1"/>
   <axis xyz="-0.0 0.0 -1.0"/>
+  <limit effort="1000.0" lower="${pi}" upper="${-pi}" velocity="100"/>
 </joint>
-<joint name="C" type="continuous">
+<joint name="${side}_mimic_1" type="continuous">
   <origin xyz="0.0 -0.06 0.006" rpy="0 0 0"/>
   <parent link="INNER_BAR_v4_1"/>
   <child link="OUTPUT_LINK_FLIPPED_v5_1"/>
   <axis xyz="-0.0 0.0 -1.0"/>
-  <mimic joint="B" multiplier="-1" offset ="0"/>
+  <mimic joint="${side}_lower_leg" multiplier="-1" offset ="0"/>
 </joint>
-<joint name="D" type="continuous">
+<joint name="${side}_mimic_2" type="continuous">
   <origin xyz="0.031 0.0 0.004" rpy="0 0 0"/>
   <parent link="OUTPUT_LINK_FLIPPED_v5_1"/>
   <child link="LONG_DRIVER_v2_1"/>
   <axis xyz="-0.0 0.0 -1.0"/>
-  <mimic joint="B" multiplier="1" offset ="0"/>
+  <mimic joint="${side}_lower_leg" multiplier="1" offset ="0"/>
 </joint>
+</xacro:macro>
 </robot>

File: qronk_description/urdf/qronk.urdf.xacro (robot description, xacro)
@@ -2,4 +2,4 @@
 <robot name="qronk" xmlns:xacro="http://www.ros.org/wiki/xacro">
     <xacro:include filename="$(find qronk_description)/urdf/qronk.xacro"/>
-    <xacro:Qronk parent="world"/>
+    <xacro:Qronk parent="base_link"/>
 </robot>

File: qronk_description/urdf/qronk.xacro (robot description, xacro)
@@ -12,12 +12,13 @@
         <link name="chassis" />
         <!-- Legs -->
-        <xacro:include filename="$(find qronk_description)/urdf/leg.xacro"/>
-        <xacro:Leg prefix="FRONT_RIGHT" />
-        <!-- ROS2 Control Tags -->
+        <xacro:include filename="$(find qronk_description)/urdf/new_leg.xacro"/>
+        <xacro:leg side="front_right" />
+        <!--
+        ROS2 Control Tags
         <xacro:include filename="$(find qronk_description)/urdf/qronk.ros2_control.xacro"/>
         <xacro:Qronk_ros2_control prefix="FRONT_RIGHT"/>
-        <!-- Gazebo Tags -->
+        Gazebo Tags
         <xacro:include filename="$(find qronk_description)/urdf/qronk.gazebo.xacro"/>
-        <xacro:Qronk_gazebo/>
+        <xacro:Qronk_gazebo/> -->
     </xacro:macro>
 </robot>

Commit message: update gazebo.launch.py to import model

File: qronk_description/urdf/new_leg.xacro (robot description, xacro)
@@ -3,5 +3,5 @@
 <xacro:include filename="$(find qronk_description)/urdf/materials.xacro" />
 <xacro:include filename="$(find qronk_description)/urdf/new_leg.trans" />
-<xacro:macro name="leg" params="side">
+<xacro:macro name="leg" params="side:=Leg parent:=world">
 <link name="SHORT_DRIVER_v3_1">
   <inertial>
@@ -86,8 +86,8 @@
 <joint name="${side}_upper_leg" type="revolute">
   <origin xyz="0.0 0.0 0.002" rpy="0 0 0"/>
-  <parent link="chassis"/>
+  <parent link="${parent}"/>
   <child link="SHORT_DRIVER_v3_1"/>
   <axis xyz="0.0 -0.0 1.0"/>
-  <limit effort="1000.0" lower="${pi}" upper="${-pi}" velocity="100"/>
+  <limit effort="1000.0" lower="${-pi}" upper="${pi}" velocity="100"/>
 </joint>
 <joint name="${side}_lower_leg" type="revolute">
@@ -96,5 +96,5 @@
   <child link="INNER_BAR_v4_1"/>
   <axis xyz="-0.0 0.0 -1.0"/>
-  <limit effort="1000.0" lower="${pi}" upper="${-pi}" velocity="100"/>
+  <limit effort="1000.0" lower="${-pi}" upper="${pi}" velocity="100"/>
 </joint>
 <joint name="${side}_mimic_1" type="continuous">

File: qronk_description/urdf/qronk.gazebo.xacro (robot description, xacro)
@@ -1,12 +1,13 @@
 <?xml version="1.0"?>
-<robot xmlns:xacro="http://www.ros.org/wiki/xacro">
-    <xacro:macro name = "Qronk_gazebo">
-    <!-- For Gazebo Sim 8 (Harmonic) with ROS2 Jazzy -->
+<robot name="qronk" xmlns:xacro="http://www.ros.org/wiki/xacro">
+    <!--Spawn Model-->
+    <xacro:include filename="$(find qronk_description)/urdf/qronk.xacro"/>
+    <xacro:Qronk parent="world"/>
     <plugin filename="gz-sim-joint-state-publisher-system" name="gz::sim::systems::JointStatePublisher">
         <topic>joint_states</topic>
         <!-- Add all the joints here -->
         <!-- <joint_name>JOINT_NAME</joint_name> -->
+        <joint_name>front_right_upper_leg</joint_name>
+        <joint_name>front_right_lower_leg</joint_name>
     </plugin>
-    <!-- plugin for IMU -->
-    </xacro:macro>
 </robot>

File: qronk_description/urdf/qronk.xacro (robot description, xacro)
@@ -4,14 +4,7 @@
         <!-- Parent (Depending on Program) -->
         <link name="${parent}" />
-        <joint name="${parent}_joint" type="fixed">
-            <parent link="${parent}" />
-            <child link="chassis" />
-            <origin xyz="0 0 0" rpy="0 0 0" />
-        </joint>
-        <!-- Chassis -->
-        <link name="chassis" />
         <!-- Legs -->
         <xacro:include filename="$(find qronk_description)/urdf/new_leg.xacro"/>
-        <xacro:leg side="front_right" />
+        <xacro:leg side="front_right" parent="${parent}"/>
         <!--
         ROS2 Control Tags
